File: AR20_ACM/ACM_pcb/01. KiCAD/MCP25625_Breakout/MCP25625_Breakoutboard/MCP25625_Breakoutboard.kicad_pcb (KiCad board)
At the start: 2 copper layers, 3 parts, among them IC1 MCP25625T-E_ML, J1 Conn_01x14, J2 Conn_01x14

Commit message: Added Gerberfiles
Other:
- board outline added: 20 x 38 mm
Changed lines of the file:
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@@
   (general
     (thickness 1.6)
-    (drawings 0)
+    (drawings 4)
     (tracks 111)
     (zones 0)
@@
   )
   (setup
-    (last_trace_width 0.35)
+    (last_trace_width 0.25)
     (user_trace_width 0.35)
     (trace_clearance 0.2)
@@
       (outputformat 1)
       (mirror false)
-      (drillshape 1)
+      (drillshape 0)
       (scaleselection 1)
-      (outputdirectory ""))
+      (outputdirectory "Gerber/V1/"))
   )
   (net 0 "")
@@
     )
   )
+  (gr_line (start 135 116) (end 135 78) (layer Edge.Cuts) (width 0.2))
+  (gr_line (start 135 116) (end 155 116) (layer Edge.Cuts) (width 0.2))
+  (gr_line (start 155 78) (end 155 116) (layer Edge.Cuts) (width 0.2))
+  (gr_line (start 135 78) (end 155 78) (layer Edge.Cuts) (width 0.2))
   (segment (start 138.61044 80.48) (end 137.67308 80.48) (width 0.35) (layer F.Cu) (net 1))
   (segment (start 143.76908 85.63864) (end 138.61044 80.48) (width 0.35) (layer F.Cu) (net 1))
