File: AR20_CPU/CPU_Breakout_Schematic/teensy4_header_breakout.sch (KiCad schematic (older format))
At the start: 54 parts, among them J1 Conn_01x14, J2 Conn_01x14, U1 GND-1

Commit message: Breakout CPU no connections added
Parts:
- removed TP? (x10): TestPoint, symbol Connector:TestPoint
Connections:
- wire segments 77 -> 67
- no-connect marks 5 -> 17
Changed lines of the file:
@@
 	0    1    1    0
 $EndComp
-$Comp
-L Connector:TestPoint TP?
-U 1 1 5DD05C93
-P 5200 3550
-F 0 "TP?" V 5200 4250 50  0000 C CNN
-F 1 "TestPoint" V 5200 3950 50  0000 C CNN
-F 2 "" H 5400 3550 50  0001 C CNN
-F 3 "~" H 5400 3550 50  0001 C CNN
-	1    5200 3550
-	0    1    1    0
-$EndComp
-Wire Wire Line
-	5200 3550 5000 3550
-$Comp
-L Connector:TestPoint TP?
-U 1 1 5DD05C9A
-P 5200 3450
-F 0 "TP?" V 5200 4150 50  0000 C CNN
-F 1 "TestPoint" V 5200 3850 50  0000 C CNN
-F 2 "" H 5400 3450 50  0001 C CNN
-F 3 "~" H 5400 3450 50  0001 C CNN
-	1    5200 3450
-	0    1    1    0
-$EndComp
 Wire Wire Line
 	5200 3650 5000 3650
-Wire Wire Line
-	5200 3450 5000 3450
-$Comp
-L Connector:TestPoint TP?
-U 1 1 5DD05CA2
-P 5200 3350
-F 0 "TP?" V 5200 4050 50  0000 C CNN
-F 1 "TestPoint" V 5200 3750 50  0000 C CNN
-F 2 "" H 5400 3350 50  0001 C CNN
-F 3 "~" H 5400 3350 50  0001 C CNN
-	1    5200 3350
-	0    1    1    0
-$EndComp
-Wire Wire Line
-	5200 3350 5000 3350
-$Comp
-L Connector:TestPoint TP?
-U 1 1 5DD05CA9
-P 5200 3250
-F 0 "TP?" V 5200 3950 50  0000 C CNN
-F 1 "TestPoint" V 5200 3650 50  0000 C CNN
-F 2 "" H 5400 3250 50  0001 C CNN
-F 3 "~" H 5400 3250 50  0001 C CNN
-	1    5200 3250
-	0    1    1    0
-$EndComp
-$Comp
-L Connector:TestPoint TP?
-U 1 1 5DD05CAF
-P 5200 3150
-F 0 "TP?" V 5200 3850 50  0000 C CNN
-F 1 "TestPoint" V 5200 3550 50  0000 C CNN
-F 2 "" H 5400 3150 50  0001 C CNN
-F 3 "~" H 5400 3150 50  0001 C CNN
-	1    5200 3150
-	0    1    1    0
-$EndComp
-Wire Wire Line
-	5200 3150 5000 3150
-$Comp
-L Connector:TestPoint TP?
-U 1 1 5DD05CB6
-P 5200 3050
-F 0 "TP?" V 5200 3750 50  0000 C CNN
-F 1 "TestPoint" V 5200 3450 50  0000 C CNN
-F 2 "" H 5400 3050 50  0001 C CNN
-F 3 "~" H 5400 3050 50  0001 C CNN
-	1    5200 3050
-	0    1    1    0
-$EndComp
-Wire Wire Line
-	5200 3250 5000 3250
-Wire Wire Line
-	5200 3050 5000 3050
-$Comp
-L Connector:TestPoint TP?
-U 1 1 5DD0A142
-P 5200 2950
-F 0 "TP?" V 5200 3650 50  0000 C CNN
-F 1 "TestPoint" V 5200 3350 50  0000 C CNN
-F 2 "" H 5400 2950 50  0001 C CNN
-F 3 "~" H 5400 2950 50  0001 C CNN
-	1    5200 2950
-	0    1    1    0
-$EndComp
-Wire Wire Line
-	5200 2950 5000 2950
-$Comp
-L Connector:TestPoint TP?
-U 1 1 5DD0A149
-P 5200 2850
-F 0 "TP?" V 5200 3550 50  0000 C CNN
-F 1 "TestPoint" V 5200 3250 50  0000 C CNN
-F 2 "" H 5400 2850 50  0001 C CNN
-F 3 "~" H 5400 2850 50  0001 C CNN
-	1    5200 2850
-	0    1    1    0
-$EndComp
-$Comp
-L Connector:TestPoint TP?
-U 1 1 5DD0A14F
-P 5200 2750
-F 0 "TP?" V 5200 3450 50  0000 C CNN
-F 1 "TestPoint" V 5200 3150 50  0000 C CNN
-F 2 "" H 5400 2750 50  0001 C CNN
-F 3 "~" H 5400 2750 50  0001 C CNN
-	1    5200 2750
-	0    1    1    0
-$EndComp
-Wire Wire Line
-	5200 2750 5000 2750
-$Comp
-L Connector:TestPoint TP?
-U 1 1 5DD0A156
-P 5200 2650
-F 0 "TP?" V 5200 3350 50  0000 C CNN
-F 1 "TestPoint" V 5200 3050 50  0000 C CNN
-F 2 "" H 5400 2650 50  0001 C CNN
-F 3 "~" H 5400 2650 50  0001 C CNN
-	1    5200 2650
-	0    1    1    0
-$EndComp
-Wire Wire Line
-	5200 2850 5000 2850
-Wire Wire Line
-	5200 2650 5000 2650
 NoConn ~ 5000 5150
 Wire Wire Line
@@
 Wire Wire Line
 	1650 4400 1600 4400
+NoConn ~ 5000 2650
+NoConn ~ 5000 2750
+NoConn ~ 5000 2850
+NoConn ~ 5000 2950
+NoConn ~ 5000 3050
+NoConn ~ 5000 3150
+NoConn ~ 5000 3250
+NoConn ~ 5000 3350
+NoConn ~ 5000 3450
+NoConn ~ 5000 3550
+NoConn ~ 4350 2250
+NoConn ~ 2000 2050
 $EndSCHEMATC

Commit message: Breakout CPU with SD card
Connections:
- wire segments 67 -> 66
- no-connect marks 17 -> 15
Changed lines of the file:
@@
 Vinn_5V
 Wire Wire Line
-	6850 4800 6850 5050
+	6850 4800 6850 4900
 Text GLabel 5550 4950 2    50   Input ~ 0
 Vinn_5V
@@
 U 1 1 5DCEE60D
 P 1700 5050
-F 0 "SW?" H 1700 5300 50  0000 C CNN
-F 1 "SW_SPST" H 1700 5200 50  0000 C CNN
+F 0 "SW?" V 1750 5300 50  0000 C CNN
+F 1 "SW_SPST" V 1650 5300 50  0000 C CNN
 F 2 "Button_Switch_SMD:SW_DIP_SPSTx01_Slide_6.7x4.1mm_W6.73mm_P2.54mm_LowProfile_JPin" H 1700 5050 50  0001 C CNN
 F 3 "~" H 1700 5050 50  0001 C CNN
@@
 L teensy4_header_breakout-cache:power_PWR_FLAG #FLG?
 U 1 1 5DD36165
-P 5500 4800
-F 0 "#FLG?" H 5500 4875 50  0001 C CNN
-F 1 "power_PWR_FLAG" H 5750 4950 50  0000 C CNN
-F 2 "" H 5500 4800 50  0001 C CNN
-F 3 "" H 5500 4800 50  0001 C CNN
-	1    5500 4800
-	1    0    0    -1
+P 6850 4900
+F 0 "#FLG?" H 6850 4975 50  0001 C CNN
+F 1 "power_PWR_FLAG" V 6850 5350 50  0000 C CNN
+F 2 "" H 6850 4900 50  0001 C CNN
+F 3 "" H 6850 4900 50  0001 C CNN
+	1    6850 4900
+	0    1    1    0
 $EndComp
 $Comp
@@
 Wire Wire Line
 	7700 5950 8050 5950
-Wire Wire Line
-	5000 4950 5500 4950
-Wire Wire Line
-	5500 4800 5500 4950
-Connection ~ 5500 4950
-Wire Wire Line
-	5500 4950 5550 4950
 Wire Wire Line
 	6050 5200 6350 5200
@@
 NoConn ~ 5000 3450
 NoConn ~ 5000 3550
-NoConn ~ 4350 2250
-NoConn ~ 2000 2050
+Connection ~ 6850 4900
+Wire Wire Line
+	6850 4900 6850 5050
+Wire Wire Line
+	5000 4950 5550 4950
 $EndSCHEMATC

Commit message: Fix
Parts:
- added J?: Micro_SD_Card, symbol Connector:Micro_SD_Card
Connections:
- wire segments 66 -> 73
Other:
- moved on the sheet: BT?, H?, JP?, R?, SW?, U?
