File: AR20_ACM/ACM_pcb/01. KiCAD/ACM_Y2020V0.1/ACM_Y2020V0.1.sch (KiCad schematic (older format))
At the start: 32 parts, among them J1 TC2030-MCP-NL, P1 Conn_02x15_Odd_Even, Q1 Q_PMOS_DGS, U1 ATmega328P-AU, U2 MCP25625-x-SS, U3 NCV890430MW50TXG, Y1 16.0Mhz

Commit message: Auto stash before merge of "master" and "origin/master"
Parts:
- removed LED1: SMLP36RGB2W3R, SMLP36RGB2W3R:SMLP36RGB2W3R, symbol ACM_Y2020V0.1-rescue:SMLP36RGB2W3R-SMLP36RGB2W3R
- removed U1: ATmega328P-AU, Package_QFP:TQFP-32_7x7mm_P0.8mm, symbol MCU_Microchip_ATmega:ATmega328P-AU
- added D3: ASMB-MTB0-0A3A2, LED_SMD:LED_Avago_PLCC4_3.2x2.8mm_CW, symbol LED:ASMB-MTB0-0A3A2
- R3: value 200 Ohm -> 290 ohm
- R4: value 290 Ohm -> 200ohm
Connections:
- wire segments 116 -> 105
Other:
- note added: "RGB krets\n"
- note removed: "LED Circuit"
- moved on the sheet: H1, J1, P1
