File: AR20_CPU/CPU_Breakout_Schematic - S.Alrawi/MCP2551.sch (KiCad schematic (older format))
At the start: 8 parts

Commit message: 4 Layers PCB is 90% finished
Parts:
- renumbered C16 to C11, H5 to H1, H6 to H2, R19 to R17, R20 to R18
Changed lines of the file:
@@
 $Descr A4 11693 8268
 encoding utf-8
-Sheet 6 6
+Sheet 3 6
 Title ""
 Date ""
@@
 	5600 2750 5600 2700
 $Comp
-L Device:C C16
+L Device:C C11
 U 1 1 5DFD4BFF
 P 5450 2900
-F 0 "C16" H 5565 2946 50  0000 L CNN
+F 0 "C11" H 5565 2946 50  0000 L CNN
 F 1 "100u" H 5565 2855 50  0000 L CNN
 F 2 "Capacitor_SMD:C_0603_1608Metric" H 5488 2750 50  0001 C CNN
@@
 $EndComp
 $Comp
-L Connector:TestPoint H5
+L Connector:TestPoint H1
 U 1 1 5DFD4C14
 P 7000 3500
-F 0 "H5" V 6954 3650 50  0000 L CNN
+F 0 "H1" V 6954 3650 50  0000 L CNN
 F 1 "CANH_out" V 7045 3650 50  0000 L CNN
 F 2 "TestPoint:TestPoint_THTPad_D1.5mm_Drill0.7mm" H 7000 3500 50  0001 C CNN
@@
 	6800 3500 7000 3500
 $Comp
-L Connector:TestPoint H6
+L Connector:TestPoint H2
 U 1 1 5DFD4C28
 P 7000 4100
-F 0 "H6" V 6954 4250 50  0000 L CNN
+F 0 "H2" V 6954 4250 50  0000 L CNN
 F 1 "CANL_out" V 7045 4250 50  0000 L CNN
 F 2 "TestPoint:TestPoint_THTPad_D1.5mm_Drill0.7mm" H 7000 4100 50  0001 C CNN
@@
 $EndComp
 $Comp
-L Device:R R20
+L Device:R R18
 U 1 1 5DFD4C2E
 P 6800 3650
-F 0 "R20" H 6900 3700 50  0000 L CNN
+F 0 "R18" H 6900 3700 50  0000 L CNN
 F 1 "120" H 6900 3600 50  0000 L CNN
 F 2 "Resistor_SMD:R_0603_1608Metric_Pad1.05x0.95mm_HandSolder" V 6730 3650 50  0001 C CNN
@@
 	5450 4100 5600 4100
 $Comp
-L Device:R R19
+L Device:R R17
 U 1 1 5DFD4C3D
 P 5300 4100
-F 0 "R19" V 5400 4100 50  0000 C CNN
+F 0 "R17" V 5400 4100 50  0000 C CNN
 F 1 "60" V 5184 4100 50  0000 C CNN
 F 2 "Resistor_SMD:R_0603_1608Metric_Pad1.05x0.95mm_HandSolder" V 5230 4100 50  0001 C CNN
