File: AR20_CPU/CPU_Breakout_Schematic - S.Alrawi/NCV890430MW50TXG.sch (KiCad schematic (older format))
At the start: 7 parts

Commit message: 4 Layers PCB is 90% finished
Parts:
- renumbered C11 to C14, C12 to C15, C13 to C16, C14 to C17, R17 to R20
Changed lines of the file:
@@
 $Descr A4 11693 8268
 encoding utf-8
-Sheet 3 6
+Sheet 5 6
 Title ""
 Date ""
@@
 $EndComp
 $Comp
-L Device:C C12
+L Device:C C15
 U 1 1 5DFC1FBC
 P 4500 3250
-F 0 "C12" H 4615 3296 50  0000 L CNN
+F 0 "C15" H 4615 3296 50  0000 L CNN
 F 1 "0.1u" H 4615 3205 50  0000 L CNN
 F 2 "Capacitor_SMD:C_0603_1608Metric" H 4538 3100 50  0001 C CNN
@@
 $EndComp
 $Comp
-L Device:C C11
+L Device:C C14
 U 1 1 5DFC1FC2
 P 4100 3250
-F 0 "C11" H 4215 3296 50  0000 L CNN
+F 0 "C14" H 4215 3296 50  0000 L CNN
 F 1 "10u" H 4215 3205 50  0000 L CNN
 F 2 "Capacitor_SMD:C_0603_1608Metric" H 4138 3100 50  0001 C CNN
@@
 $EndComp
 $Comp
-L Device:C C13
+L Device:C C16
 U 1 1 5DFC1FC8
 P 7100 3200
-F 0 "C13" H 7215 3246 50  0000 L CNN
+F 0 "C16" H 7215 3246 50  0000 L CNN
 F 1 "0.1u" H 7215 3155 50  0000 L CNN
 F 2 "Capacitor_SMD:C_0603_1608Metric" H 7138 3050 50  0001 C CNN
@@
 $EndComp
 $Comp
-L Device:C C14
+L Device:C C17
 U 1 1 5DFC1FCE
 P 7500 3200
-F 0 "C14" H 7615 3246 50  0000 L CNN
+F 0 "C17" H 7615 3246 50  0000 L CNN
 F 1 "10u" H 7615 3155 50  0000 L CNN
 F 2 "Capacitor_SMD:C_0603_1608Metric" H 7538 3050 50  0001 C CNN
@@
 Vinn_5V
 $Comp
-L Device:R R17
+L Device:R R20
 U 1 1 5DFC1FFA
 P 4900 3200
-F 0 "R17" H 4700 3300 50  0000 L CNN
+F 0 "R20" H 4700 3300 50  0000 L CNN
 F 1 "10k" H 4950 3300 50  0000 L CNN
 F 2 "Resistor_SMD:R_0603_1608Metric" V 4830 3200 50  0001 C CNN
