File: AR20_CPU/CPU_Breakout_Schematic - S.Alrawi/teensy4_header_breakout.sch (KiCad schematic (older format))
At the start: 11 parts, among them J1 Conn_2Rows-34Pins, J3 Micro_SD_Card, SW1 SW_SPST, U1 Teensy_pins, U2 MCP2551-I-SN

Commit message: Edited library
Parts:
- removed J1: Conn_2Rows-34Pins, Teensy_Footprint_Library:PINS_IO_TEENSY, symbol BreakoutBoardTeensy:Conn_2Rows-34Pins
- added C1, C2, C4, C5: 1.5n, Capacitor_SMD:C_0603_1608Metric, symbol Device:C
- added C3: C, Capacitor_SMD:C_0603_1608Metric, symbol Device:C
- added C6, C9: 10u, Capacitor_SMD:C_0603_1608Metric, symbol Device:C
- added C7, C8: 0.1u, Capacitor_SMD:C_0603_1608Metric, symbol Device:C
- added D1, D2, D3, D4: 3V, Diode_SMD:D_0603_1608Metric, symbol Device:D_Zener
- added IC1: LM324DRG3, Package_SO:SOIC-14_3.9x8.7mm_P1.27mm, symbol BreakoutBoardTeensy:LM324DRG3
- added IC2: NCV890430MW50TXG, Package_DFN_QFN:DFN-8-1EP_3x3mm_P0.65mm_EP1.7x2.05mm, symbol NCV890430MW50TXG:NCV890430MW50TXG
- added J?: Conn_01x17, symbol BreakoutBoardTeensy:Conn_01x17
- added J?: Conn_01x15, symbol BreakoutBoardTeensy:Conn_01x15
- added L1: 2.2u, Inductor_SMD:L_0603_1608Metric, symbol Device:L
- added R10, R4, R6, R8: 20k, Resistor_SMD:R_0603_1608Metric, symbol Device:R
- added R11, R3, R5, R7, R9: 10k, Resistor_SMD:R_0603_1608Metric, symbol Device:R
- H1, H2: symbol Mechanical:MountingHole_Pad -> Connector:TestPoint
Connections:
- net labels added: 12V_IN, IN1+, IN2+, IN3+, IN4+, Out1, Out2, Out3, Out4, Sensor_Input_1, Sensor_Input_2, Sensor_Input_3, Sensor_Input_4
- net labels removed: 18_A4, 19_A5, 20_A6, 21_A7, PROGRAMM
- wire segments 107 -> 199
- no-connect marks 3 -> 4
Other:
- note added: "From sensor"
- note added: "To analog pin"
- moved on the sheet: J3, U1

Commit message: Edited the layout
Parts:
- removed J?: Conn_01x17, symbol BreakoutBoardTeensy:Conn_01x17
- removed J?: Conn_01x15, symbol BreakoutBoardTeensy:Conn_01x15
- added C10: 1.5n, Capacitor_SMD:C_0603_1608Metric, symbol Device:C
- added GND1: GND, TestPoint:TestPoint_THTPad_D1.5mm_Drill0.7mm, symbol Connector:TestPoint
- added J1: MX34_36_pins, Teensy_Footprint_Library:Connector_MX34_36pins, symbol teensy4_header_breakout-cache:MX34_36_pins
- added JP2, JP3, JP4, JP5: SJ_Open, Jumper:SolderJumper-2_P1.3mm_Open_RoundedPad1.0x1.5mm, symbol Jumper:SolderJumper_2_Open
- added MX34_Housing1: MX34_Housing, Teensy_Footprint_Library:Housing_3pins, symbol BreakoutBoardTeensy:MX34_Housing
- added R12: 20k, Resistor_SMD:R_0603_1608Metric, symbol Device:R
- C2: value 1.5n -> 10u
- R6: value 20k -> 10k
- renumbered U2 to CANmodule1, IC1 to LM324, J3 to SDcard1, IC2 to SWReg_NVC1, U1 to Teensy4.0
Connections:
- net labels removed: GND_1, GND_BATT
- wire segments 199 -> 206
- no-connect marks 4 -> 2

Commit message: Edited to 4 layers
Parts:
- removed BT1: 2.7V, Battery:BatteryHolder_Keystone_3034_1x20mm, symbol Device:Battery_Cell
- removed C1, C10, C4, C5: 1.5n, Capacitor_SMD:C_0603_1608Metric, symbol Device:C
- removed C2, C6, C9: 10u, Capacitor_SMD:C_0603_1608Metric, symbol Device:C
- removed C3: C, Capacitor_SMD:C_0603_1608Metric, symbol Device:C
- removed C7, C8: 0.1u, Capacitor_SMD:C_0603_1608Metric, symbol Device:C
- removed CANmodule1: MCP2551-I-SN, Package_SO:SOIC-8_3.9x4.9mm_P1.27mm, symbol Interface_CAN_LIN:MCP2551-I-SN
- removed D1, D2, D3, D4: 3V, Diode_SMD:D_0603_1608Metric, symbol Device:D_Zener
- removed GND1: GND, TestPoint:TestPoint_THTPad_D1.5mm_Drill0.7mm, symbol Connector:TestPoint
- removed H1: CANH_out, TestPoint:TestPoint_THTPad_D1.5mm_Drill0.7mm, symbol Connector:TestPoint
- removed H2: CANL_out, TestPoint:TestPoint_THTPad_D1.5mm_Drill0.7mm, symbol Connector:TestPoint
- removed J1: MX34_36_pins, Teensy_Footprint_Library:Connector_MX34_36pins, symbol teensy4_header_breakout-cache:MX34_36_pins
- removed JP1: SolderJumper_2_Open, Jumper:SolderJumper-2_P1.3mm_Open_RoundedPad1.0x1.5mm, symbol Jumper:SolderJumper_2_Open
- removed JP2, JP3, JP4, JP5: SJ_Open, Jumper:SolderJumper-2_P1.3mm_Open_RoundedPad1.0x1.5mm, symbol Jumper:SolderJumper_2_Open
- removed L1: 2.2u, Inductor_SMD:L_0603_1608Metric, symbol Device:L
- removed LM324: LM324DRG3, Package_SO:SOIC-14_3.9x8.7mm_P1.27mm, symbol BreakoutBoardTeensy:LM324DRG3
- removed MX34_Housing1: MX34_Housing, Teensy_Footprint_Library:Housing_3pins, symbol BreakoutBoardTeensy:MX34_Housing
- removed R1: 60, Resistor_SMD:R_0603_1608Metric_Pad1.05x0.95mm_HandSolder, symbol Device:R
- removed R10, R12, R4, R8: 20k, Resistor_SMD:R_0603_1608Metric, symbol Device:R
- removed R11, R3, R5, R6, R7, R9: 10k, Resistor_SMD:R_0603_1608Metric, symbol Device:R
- removed R2: 120, Resistor_SMD:R_0603_1608Metric_Pad1.05x0.95mm_HandSolder, symbol Device:R
- removed SDcard1: Micro_SD_Card, Connector_Card:microSD_HC_Hirose_DM3D-SF, symbol Connector:Micro_SD_Card
- removed SW1: SW_SPST, Button_Switch_SMD:SW_DIP_SPSTx01_Slide_6.7x4.1mm_W6.73mm_P2.54mm_LowProfile_JPin, symbol Switch:SW_SPST
- removed SWReg_NVC1: NCV890430MW50TXG, Package_DFN_QFN:DFN-8-1EP_3x3mm_P0.65mm_EP1.7x2.05mm, symbol NCV890430MW50TXG:NCV890430MW50TXG
- removed Teensy4.0: Teensy_pins, Teensy_Footprint_Library:Teensy_40_footprint, symbol BreakoutBoardTeensy:Teensy_pins
Connections:
- no-connect marks 2 -> 0
Other:
- note removed: "From sensor"
- note removed: "To analog pin"
