File: AR20_CPU/CPU_Breakout/teensy4_header_breakout.sch (KiCad schematic (older format))
At the start: 0 parts

Commit message: E
Changed lines of the file:
@@
 $EndDescr
 $Sheet
-S 1700 5550 1150 950
+S 2400 5250 1150 950
 U 5DE81E30
 F0 "LM324" 50
