File: AR20_CPU/CPU_Breakout/MCP2551.sch (KiCad schematic (older format))
At the start: 8 parts

Commit message: E
Parts:
- C11: value 100u -> .1u
Connections:
- net 22_CTX1 renamed 31_CTX3
- net 23_CRX1 renamed 30_CRX3
Changed lines of the file:
@@
 P 5450 2900
 F 0 "C11" H 5565 2946 50  0000 L CNN
-F 1 "100u" H 5565 2855 50  0000 L CNN
+F 1 ".1u" H 5565 2855 50  0000 L CNN
 F 2 "Capacitor_SMD:C_0603_1608Metric" H 5488 2750 50  0001 C CNN
 F 3 "~" H 5450 2900 50  0001 C CNN
@@
 Wire Wire Line
 	5100 3350 5100 3400
-Wire Wire Line
-	4800 3350 5100 3350
 Wire Wire Line
 	6450 4100 6800 4100
@@
 	1    0    0    -1
 $EndComp
-Text GLabel 4800 3550 0    50   Input ~ 0
-23_CRX1
-Text GLabel 4800 3350 0    50   Input ~ 0
-22_CTX1
 $Comp
 L Interface_CAN_LIN:MCP2551-I-SN CANmodule1
@@
 Text GLabel 5200 2900 0    50   Input ~ 0
 Ground
+Text GLabel 4800 3550 0    50   Input ~ 0
+30_CRX3
+Text GLabel 4800 3350 0    50   Input ~ 0
+31_CTX3
+Wire Wire Line
+	4800 3350 5100 3350
 $EndSCHEMATC

Commit message: Edit pads
Parts:
- GND1, H1, H2: footprint TestPoint:TestPoint_THTPad_D1.5mm_Drill0.7mm -> TestPoint:TestPoint_THTPad_D2.0mm_Drill1.0mm
Changed lines of the file:
@@
 F 0 "GND1" V 5654 4350 50  0000 L CNN
 F 1 "GND" V 5745 4350 50  0000 L CNN
-F 2 "TestPoint:TestPoint_THTPad_D1.5mm_Drill0.7mm" H 5700 4200 50  0001 C CNN
+F 2 "TestPoint:TestPoint_THTPad_D2.0mm_Drill1.0mm" H 5700 4200 50  0001 C CNN
 F 3 "~" H 5700 4200 50  0001 C CNN
 	1    5700 4200
@@
 F 0 "H1" V 6954 3650 50  0000 L CNN
 F 1 "CANH_out" V 7045 3650 50  0000 L CNN
-F 2 "TestPoint:TestPoint_THTPad_D1.5mm_Drill0.7mm" H 7000 3500 50  0001 C CNN
+F 2 "TestPoint:TestPoint_THTPad_D2.0mm_Drill1.0mm" H 7000 3500 50  0001 C CNN
 F 3 "~" H 7000 3500 50  0001 C CNN
 	1    7000 3500
@@
 F 0 "H2" V 6954 4250 50  0000 L CNN
 F 1 "CANL_out" V 7045 4250 50  0000 L CNN
-F 2 "TestPoint:TestPoint_THTPad_D1.5mm_Drill0.7mm" H 7000 4100 50  0001 C CNN
+F 2 "TestPoint:TestPoint_THTPad_D2.0mm_Drill1.0mm" H 7000 4100 50  0001 C CNN
 F 3 "~" H 7000 4100 50  0001 C CNN
 	1    7000 4100
