File: AR20_ACM/ACM_pcb/01. KiCAD/ACM_2020_Mohammad_edition 3/ACM_Y2020V0.1.kicad_pcb (KiCad board)
At the start: 2 copper layers, 32 parts, among them J1 TC2030-MCP-NL, P1 Conn_02x15_Odd_Even, Q1 Q_PMOS_DGS, U1 ATmega328P-AU, U2 MCP25625-x-SS, U3 NCV890430MW50TXG, Y1 16.0Mhz

Commit message: ready pcb ACM
Parts:
- moved R1 5.06 mm to (70.4, 79.9)
- moved D1 3.60 mm to (76.5, 89.1)
- moved R2 3.55 mm to (74.0, 89.1)
- moved Q1 3.52 mm to (76.1, 86.6)
- moved D3 3.52 mm to (66.6, 78.8), turned to 90 degrees
- moved D2 3.50 mm to (73.5, 86.6)
- moved F1 3.50 mm to (78.6, 85.8)
- moved J1 0.91 mm to (69.4, 86.2)
- moved R5 0.08 mm to (70.4, 77.7)
- moved R3 0.06 mm to (69.5, 77.0)
Connections:
- net Net-(P1-Pad10) renamed /U-Pin10
- net Net-(P1-Pad24) renamed /U-Pin24
- net Net-(P1-Pad26) renamed /U-Pin26
- net Net-(P1-Pad28) renamed /U-Pin28
- net Net-(P1-Pad30) renamed /U-Pin30
- net Net-(P1-Pad5) renamed /U-Pin5
- P1 pad 11: Net-(P1-Pad11) -> /SCK
- P1 pad 12: Net-(P1-Pad12) -> /U-Pin12
- P1 pad 13: Net-(P1-Pad13) -> /MISO
- P1 pad 14: Net-(P1-Pad14) -> /U-Pin14
- P1 pad 15: Net-(P1-Pad15) -> /MOSI
- P1 pad 2: Net-(P1-Pad2) -> /U-Pin2
- P1 pad 20: Net-(P1-Pad20) -> /U-Pin20
- P1 pad 22: Net-(P1-Pad22) -> /U-Pin22
- P1 pad 23: Net-(P1-Pad23) -> /U-Pin23
- P1 pad 4: Net-(P1-Pad4) -> /U-Pin4
- P1 pad 6: Net-(P1-Pad6) -> /U-Pin6
- P1 pad 8: Net-(P1-Pad8) -> /U-Pin8
- P1 pad 9: Net-(P1-Pad9) -> /CAN_CS
Routing:
- net GND: track 70.5 -> 46.3 mm, vias 4 -> 5
- net +5V: track 17.9 -> 28.1 mm
- net Net-(D3-Pad3): track 11.9 -> 2.09 mm
- net Net-(D3-Pad2): track 2.56 -> 9.91 mm
- net /U-Pin2: track 0.00 -> 7.25 mm, vias 0 -> 1
- net /U-Pin4: track 0.00 -> 6.59 mm, vias 0 -> 1
- net /U-Pin6: track 0.00 -> 6.17 mm, vias 0 -> 1
- net +12V_Safe: track 10.9 -> 16.9 mm
- net /U-Pin8: track 0.00 -> 5.51 mm, vias 0 -> 1
- net /U-Pin23: track 0.00 -> 4.19 mm, vias 0 -> 1
- net /U-Pin12: track 0.00 -> 4.16 mm, vias 0 -> 1
- net /U-Pin14: track 0.00 -> 3.69 mm, vias 0 -> 1
- net /U-Pin22: track 0.00 -> 3.41 mm, vias 0 -> 1
- net /U-Pin20: track 0.00 -> 3.00 mm, vias 0 -> 1
- net /MISO: track 17.9 -> 20.4 mm
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