File: AR20_ACM/ACM_pcb/01. KiCAD/ACM Breakout/ACM Breakout/ACM Breakout.kicad_pcb (KiCad board)
At the start: 2 copper layers, 3 parts, among them J1 Conn_01x15_Male, J2 Conn_01x15_Male, U1 ACM_2020

Commit message: Pad to close to pad issue
Routing:
- net /Pin1: track 9.39 -> 0.00 mm
Other:
- rule trace_min: 0.2 -> 0.127
- rule via_min_size: 0.4 -> 0.6
Changed lines of the file:
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@@
     (thickness 1.6)
     (drawings 0)
-    (tracks 107)
+    (tracks 102)
     (zones 0)
     (modules 3)
@@
   )
   (setup
-    (last_trace_width 0.254)
+    (last_trace_width 0.25)
     (user_trace_width 0.254)
     (trace_clearance 0.2)
     (zone_clearance 0.508)
     (zone_45_only no)
-    (trace_min 0.2)
+    (trace_min 0.127)
     (via_size 0.8)
     (via_drill 0.4)
-    (via_min_size 0.4)
+    (via_min_size 0.6)
     (via_min_drill 0.3)
     (uvia_size 0.3)
@@
     (solder_mask_min_width 0.25)
     (aux_axis_origin 0 0)
-    (visible_elements FFFFFF7F)
+    (visible_elements 7FFFFFFF)
     (pcbplotparams
       (layerselection 0x010fc_ffffffff)
@@
     )
   )
-  (segment (start 11.850001 -0.470001) (end 12.7 -1.32) (width 0.254) (layer F.Cu) (net 1))
-  (segment (start 8.476 2.904) (end 11.850001 -0.470001) (width 0.254) (layer F.Cu) (net 1))
-  (segment (start 6.2814 2.904) (end 8.476 2.904) (width 0.254) (layer F.Cu) (net 1))
-  (segment (start 5.7524 2.375) (end 6.2814 2.904) (width 0.254) (layer F.Cu) (net 1))
-  (segment (start 5.7524 1.9) (end 5.7524 2.375) (width 0.254) (layer F.Cu) (net 1))
   (segment (start 11.850001 2.069999) (end 12.7 1.22) (width 0.254) (layer F.Cu) (net 2))
   (segment (start 10.237 3.683) (end 11.850001 2.069999) (width 0.254) (layer F.Cu) (net 2))
