File: AR20_ACM/ACM_pcb/01. KiCAD/ACM Breakout/ACM Breakout/ACM Breakout.sch (KiCad schematic (older format))
At the start: 3 parts, among them J1 Conn_01x15_Male, J2 Conn_01x15_Male, U1 ACM_2020

Commit message: Generated gerber for breakout board
Parts:
- U1: footprint ACM_2020_Footprintandsymbol:ACM_2020Footprint -> ACM_2020_Footprintandsymbol:ACM_2020_Footprint_wo_silk
Changed lines of the file:
@@
 F 0 "U1" H 5625 7240 50  0000 C CNN
 F 1 "ACM_2020" H 5625 7149 50  0000 C CNN
-F 2 "ACM_2020_Footprintandsymbol:ACM_2020Footprint" H 5600 4675 50  0001 C CNN
+F 2 "ACM_2020_Footprintandsymbol:ACM_2020_Footprint_wo_silk" H 5600 4675 50  0001 C CNN
 F 3 "" H 5600 4675 50  0001 C CNN
 	1    5600 4675
