File: AR20_CPU/CPU_Breakout_2_layers_V2.0/MCP2551.sch (KiCad schematic (older format))
At the start: 8 parts

Commit message: V2.0 Teensy Breakout Board
Parts:
- removed GND1: GND, TestPoint:TestPoint_THTPad_D2.0mm_Drill1.0mm, symbol Connector:TestPoint
- removed H1: CANH_out, TestPoint:TestPoint_THTPad_D2.0mm_Drill1.0mm, symbol Connector:TestPoint
- removed H2: CANL_out, TestPoint:TestPoint_THTPad_D2.0mm_Drill1.0mm, symbol Connector:TestPoint
- R17: value 60 -> 68
Connections:
- net labels added: CANH, CANL
- wire segments 22 -> 19
Changed lines of the file:
@@
 Text GLabel 5600 2700 1    50   Input ~ 0
 Vinn_5V
-Wire Wire Line
-	5700 4200 5600 4200
-Connection ~ 5700 4200
-$Comp
-L Connector:TestPoint GND1
-U 1 1 5DFD4C0E
-P 5700 4200
-F 0 "GND1" V 5654 4350 50  0000 L CNN
-F 1 "GND" V 5745 4350 50  0000 L CNN
-F 2 "TestPoint:TestPoint_THTPad_D2.0mm_Drill1.0mm" H 5700 4200 50  0001 C CNN
-F 3 "~" H 5700 4200 50  0001 C CNN
-	1    5700 4200
-	1    0    0    -1
-$EndComp
-$Comp
-L Connector:TestPoint H1
-U 1 1 5DFD4C14
-P 7000 3500
-F 0 "H1" V 6954 3650 50  0000 L CNN
-F 1 "CANH_out" V 7045 3650 50  0000 L CNN
-F 2 "TestPoint:TestPoint_THTPad_D2.0mm_Drill1.0mm" H 7000 3500 50  0001 C CNN
-F 3 "~" H 7000 3500 50  0001 C CNN
-	1    7000 3500
-	0    1    1    0
-$EndComp
 NoConn ~ 5100 3700
 Wire Wire Line
@@
 Wire Wire Line
 	6450 3700 6450 4100
-Connection ~ 6800 4100
-Wire Wire Line
-	6800 4100 7000 4100
 Wire Wire Line
 	6100 3500 6800 3500
-Connection ~ 6800 3500
-Wire Wire Line
-	6800 3500 7000 3500
-$Comp
-L Connector:TestPoint H2
-U 1 1 5DFD4C28
-P 7000 4100
-F 0 "H2" V 6954 4250 50  0000 L CNN
-F 1 "CANL_out" V 7045 4250 50  0000 L CNN
-F 2 "TestPoint:TestPoint_THTPad_D2.0mm_Drill1.0mm" H 7000 4100 50  0001 C CNN
-F 3 "~" H 7000 4100 50  0001 C CNN
-	1    7000 4100
-	0    1    1    0
-$EndComp
-$Comp
-L Device:R R18
-U 1 1 5DFD4C2E
-P 6800 3650
-F 0 "R18" H 6900 3700 50  0000 L CNN
-F 1 "120" H 6900 3600 50  0000 L CNN
-F 2 "Resistor_SMD:R_0603_1608Metric_Pad1.05x0.95mm_HandSolder" V 6730 3650 50  0001 C CNN
-F 3 "~" H 6800 3650 50  0001 C CNN
-	1    6800 3650
-	1    0    0    -1
-$EndComp
 $Comp
 L Jumper:SolderJumper_2_Open JP9
@@
 P 5300 4100
 F 0 "R17" V 5400 4100 50  0000 C CNN
-F 1 "60" V 5184 4100 50  0000 C CNN
+F 1 "68" V 5184 4100 50  0000 C CNN
 F 2 "Resistor_SMD:R_0603_1608Metric_Pad1.05x0.95mm_HandSolder" V 5230 4100 50  0001 C CNN
 F 3 "~" H 5300 4100 50  0001 C CNN
@@
 	5600 4200 5600 4250
 Connection ~ 5600 4200
-Wire Wire Line
-	5750 4200 5700 4200
 Text GLabel 5750 4200 2    50   Input ~ 0
 Ground
@@
 Wire Wire Line
 	4800 3350 5100 3350
+Text GLabel 6700 4100 3    50   Input ~ 0
+CANL
+Text GLabel 6750 3500 1    50   Input ~ 0
+CANH
+$Comp
+L Device:R R18
+U 1 1 5DFD4C2E
+P 6800 3650
+F 0 "R18" H 6900 3700 50  0000 L CNN
+F 1 "120" H 6900 3600 50  0000 L CNN
+F 2 "Resistor_SMD:R_0603_1608Metric_Pad1.05x0.95mm_HandSolder" V 6730 3650 50  0001 C CNN
+F 3 "~" H 6800 3650 50  0001 C CNN
+	1    6800 3650
+	1    0    0    -1
+$EndComp
+Wire Wire Line
+	5600 4200 5750 4200
 $EndSCHEMATC
