File: AR20_CPU/CPU_Breakout_2_layers_V2.0/teensy4_header_breakout.kicad_pcb (KiCad board)
At the start: 2 copper layers, 65 x 80 mm, 66 parts, among them SW1 SW_Push_Dual, T4 BreakoutBoardTeensy_Teensy_pi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, U1 S8211-46R

Commit message: Edited
Parts:
- moved SW1 0.54 mm to (171.5, 109.2)
Connections:
- MX1 pad 25: Ground -> 26_A12
- T4 pad 37: (no net) -> 26_A12
Routing:
- net 26_A12: track 0.00 -> 27.2 mm, vias 0 -> 1
- net Ground: track 116.2 -> 123.9 mm
- net 29_TX7: track 30.8 -> 35.4 mm
- net CANL: track 23.8 -> 22.7 mm
- net ON_OFF: track 25.6 -> 24.6 mm
Other:
- board text added: "T4AR20V2.0"
- board text removed: "T4.1AR20"

Commit message: Push button edited
Parts:
- added C12: 10u, Capacitor_SMD:C_0603_1608Metric_Pad1.05x0.95mm_HandSolder, F.Cu at (170.1, 100.3)
- added SW2: SW_Push, Button_Switch_SMD:SW_SPST_B3U-1000P, F.Cu at (172.0, 107.0)
- SW1: value SW_Push_Dual -> SW_Push; footprint Button_Switch_SMD:SW_SPST_B3S-1000 -> Button_Switch_SMD:SW_SPST_B3U-1000P
- moved SW1 1.72 mm to (171.9, 110.9), turned to 0 degrees
Connections:
- SW1 pad 1: Ground -> Program
- SW1 pad 2: ON_OFF -> Ground
- T4 pad 32: (no net) -> Program
Routing:
- net ON_OFF: track 24.6 -> 11.1 mm
- net Program: track 0.00 -> 12.1 mm, vias 0 -> 1
- net 12_MISO: track 35.4 -> 36.0 mm
- net 3.3V: track 46.4 -> 46.9 mm

Commit message: Edited
Parts:
- added C13: 10u, Capacitor_SMD:C_0603_1608Metric, F.Cu at (128.2, 104.8)
Routing:
- net Vinn_5V: track 30.1 -> 32.4 mm
- net Ground: track 124.0 -> 126.3 mm
Changed lines of the file:
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@@
     (thickness 1.6)
     (drawings 7)
-    (tracks 725)
+    (tracks 729)
     (zones 0)
-    (modules 68)
+    (modules 69)
     (nets 73)
   )
@@
     (add_net "Net-(CANmodule1-Pad5)")
     (add_net "Net-(CANmodule1-Pad8)")
-    (add_net "Net-(JP10-Pad1)")
-    (add_net "Net-(JP10-Pad2)")
     (add_net "Net-(JP9-Pad1)")
     (add_net "Net-(L1-Pad1)")
@@
     (add_net Vinn_5V)
   )
+  (module Capacitor_SMD:C_0603_1608Metric (layer Front_GND)
+    (at 128.23952 104.81818 180)
+    (descr "Capacitor SMD 0603 (1608 Metric), square (rectangular) end terminal, IPC_7351 nominal, (Body size source: http://www.tortai-tech.com/upload/download/2011102023233369053.pdf), generated with kicad-footprint-generator")
+    (tags capacitor)
+    (attr smd)
+    (fp_text reference C13 (at 0 -1.43) (layer F.SilkS)
+      (effects (font (size 1 1) (thickness 0.15)))
+    )
+    (fp_text value 10u (at 0 1.43) (layer F.Fab)
+      (effects (font (size 1 1) (thickness 0.15)))
+    )
+    (fp_text user %R (at 0 0) (layer F.Fab)
+      (effects (font (size 0.4 0.4) (thickness 0.06)))
+    )
+    (fp_line (start 1.48 0.73) (end -1.48 0.73) (layer F.CrtYd) (width 0.05))
+    (fp_line (start 1.48 -0.73) (end 1.48 0.73) (layer F.CrtYd) (width 0.05))
+    (fp_line (start -1.48 -0.73) (end 1.48 -0.73) (layer F.CrtYd) (width 0.05))
+    (fp_line (start -1.48 0.73) (end -1.48 -0.73) (layer F.CrtYd) (width 0.05))
+    (fp_line (start -0.162779 0.51) (end 0.162779 0.51) (layer F.SilkS) (width 0.12))
+    (fp_line (start -0.162779 -0.51) (end 0.162779 -0.51) (layer F.SilkS) (width 0.12))
+    (fp_line (start 0.8 0.4) (end -0.8 0.4) (layer F.Fab) (width 0.1))
+    (fp_line (start 0.8 -0.4) (end 0.8 0.4) (layer F.Fab) (width 0.1))
+    (fp_line (start -0.8 -0.4) (end 0.8 -0.4) (layer F.Fab) (width 0.1))
+    (fp_line (start -0.8 0.4) (end -0.8 -0.4) (layer F.Fab) (width 0.1))
+    (pad 2 smd roundrect (at 0.7875 0 180) (size 0.875 0.95) (layers Front_GND F.Paste F.Mask) (roundrect_rratio 0.25)
+      (net 4 Vinn_5V))
+    (pad 1 smd roundrect (at -0.7875 0 180) (size 0.875 0.95) (layers Front_GND F.Paste F.Mask) (roundrect_rratio 0.25)
+      (net 1 Ground))
+    (model ${KISYS3DMOD}/Capacitor_SMD.3dshapes/C_0603_1608Metric.wrl
+      (at (xyz 0 0 0))
+      (scale (xyz 1 1 1))
+      (rotate (xyz 0 0 0))
+    )
+  )
   (module Capacitor_SMD:C_0603_1608Metric_Pad1.05x0.95mm_HandSolder (layer Front_GND)
     (at 170.05554 100.3427 90)
@@
   (segment (start 170.79338 99.4677) (end 171.16806 99.09302) (width 0.25) (layer Front_GND) (net 1))
   (segment (start 170.05554 99.4677) (end 170.79338 99.4677) (width 0.25) (layer Front_GND) (net 1))
+  (segment (start 129.02702 103.11628) (end 129.45618 102.68712) (width 0.5) (layer Front_GND) (net 1))
+  (segment (start 129.02702 104.81818) (end 129.02702 103.11628) (width 0.5) (layer Front_GND) (net 1))
   (via (at 161.03854 111.59744) (size 1) (drill 0.5) (layers Front_GND Back_GND) (net 2))
   (segment (start 161.39922 111.95812) (end 161.03854 111.59744) (width 0.25) (layer Front_GND) (net 2))
@@
   (segment (start 125.14344 134.15536) (end 125.4125 134.42442) (width 0.5) (layer Front_GND) (net 4))
   (segment (start 125.14344 130.16738) (end 125.14344 134.15536) (width 0.5) (layer Front_GND) (net 4))
+  (segment (start 127.45202 103.22296) (end 126.91618 102.68712) (width 0.5) (layer Front_GND) (net 4))
+  (segment (start 127.45202 104.81818) (end 127.45202 103.22296) (width 0.5) (layer Front_GND) (net 4))
   (via (at 165.5064 103.0732) (size 1) (drill 0.5) (layers Front_GND Back_GND) (net 5))
   (via (at 165.36465 115.59286) (size 1) (drill 0.5) (layers Front_GND Back_GND) (net 5))
