File: Teensy_CPU_CircuitBoard/CPU_Breakout_2_layers_V2.0/teensy4_header_breakout.kicad_pcb (KiCad board)
At the start: 2 copper layers, 65 x 80 mm, 69 parts, among them SW1 SW_Push, SW2 SW_Push, T4 BreakoutBoardTeensy_Teensy_pi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, U1 S8211-46R

Commit message: Start of V3 STM32
Imported symbols/footprints ...
Parts:
- removed C14, C17: 10u, Capacitor_SMD:C_0603_1608Metric
- removed C15, C16: 0.1u, Capacitor_SMD:C_0603_1608Metric
- removed L1: 2.2u, Inductor_SMD:L_0603_1608Metric
- removed R20: 10k, Resistor_SMD:R_0603_1608Metric
- removed SWReg_NVC1: NCV890430MW50TXG, Package_DFN_QFN:DFN-8-1EP_3x3mm_P0.65mm_EP1.7x2.05mm
- added D9: D_RPP_Input_PMEG4010EGWX, Teensy_Footprint_Library:D_RPP_PMEG4010EGWX, F.Cu at (207.0, 76.2)
- added PS1: TEL_5-1211, Teensy_Footprint_Library:TEL51211, F.Cu at (194.6, 98.0)

Commit message: PCB trace 1.0V
Har ikke lagt til spenningsforsyning til sensorene eller GND. Dessuten har jeg satt connectoren feil vei
Parts:
- removed C12: 10u, Capacitor_SMD:C_0603_1608Metric_Pad1.05x0.95mm_HandSolder
- removed C13, C18: 10u, Capacitor_SMD:C_0603_1608Metric
- removed CANmodule1: MCP2551-I-SN, Package_SO:SOIC-8_3.9x4.9mm_P1.27mm
- removed D7, D8: 3V, Diode_SMD:D_0603_1608Metric
- removed D9: D_RPP_Input_PMEG4010EGWX, Teensy_Footprint_Library:D_RPP_PMEG4010EGWX
- removed H4, H5, H6, H7: MountingHole, MountingHole:MountingHole_2.5mm_Pad
- removed JP1, JP2, JP3, JP4, JP5, JP6, JP7, JP8: SJ_Open, Jumper:SolderJumper-2_P1.3mm_Open_RoundedPad1.0x1.5mm
- removed JP9: SolderJumper_2_Open, Jumper:SolderJumper-2_P1.3mm_Open_RoundedPad1.0x1.5mm
- removed LM1, LM2: LM324DRG3, Package_SO:SOIC-14_3.9x8.7mm_P1.27mm
- removed R10, R12, R14, R16: 20k, Resistor_SMD:R_0603_1608Metric
- removed R11, R13, R15, R9: 10k, Resistor_SMD:R_0603_1608Metric
- removed R17: 68, Resistor_SMD:R_0603_1608Metric_Pad1.05x0.95mm_HandSolder
- removed R18: 120, Resistor_SMD:R_0603_1608Metric_Pad1.05x0.95mm_HandSolder
- removed SW1, SW2: SW_Push, Button_Switch_SMD:SW_SPST_B3U-1000P
- removed T4: BreakoutBoardTeensy_Teensy_pins, Teensy_Footprint_Library:Teensy_40_footprint
- added F1: Polyfuse_Small, Resistor_SMD:R_1210_3225Metric_Pad1.30x2.65mm_HandSolder, F.Cu at (238.0, 32.5)
- added U2: NUCLEO-H745ZI-Q, Teensy_Footprint_Library:MODULE_NUCLEO-F429ZI, F.Cu at (99.6, 106.2)
- added U3: MCP2542WFDxMF, Package_DFN_QFN:DFN-8-1EP_3x3mm_P0.65mm_EP1.55x2.4mm, F.Cu at (192.0, 93.5)
- added Z1: 1SMB5930BT3G, Teensy_Footprint_Library:DIOM5436X247N, F.Cu at (233.9, 39.6)
- C1, C2, C4, C5: value 1.5n -> 15n
- C10, C6, C7, C9: value 1.5n -> 10uF
- C11: value .1u -> 10uF; moved to F.Cu
- C3: value C -> 15n
- C8: value C -> 10uF
- D1: value 3V -> D_Schottky_MBR0520LT1G; footprint Diode_SMD:D_0603_1608Metric -> Teensy_Footprint_Library:D_SOD-123-MBR0520LT1G
- D2, D3, D4, D5, D6: value 3V -> D_Zener_MM3Z3V6T1G; footprint Diode_SMD:D_0603_1608Metric -> Teensy_Footprint_Library:D_0603_MM3Z3V6T1G
- R2, R4: value 20k -> 10k
- R7: value 10k -> 120; footprint Resistor_SMD:R_0603_1608Metric -> Resistor_SMD:R_0603_1608Metric_Pad0.98x0.95mm_HandSolder
- R8: value 20k -> 120; footprint Resistor_SMD:R_0603_1608Metric -> Resistor_SMD:R_0603_1608Metric_Pad0.98x0.95mm_HandSolder
- SDcard1: footprint Connector_Card:microSD_HC_Hirose_DM3D-SF -> Teensy_Footprint_Library:Molex_502774-0891; moved to F.Cu
- U1: value S8211-46R -> MCP2542WFDxMF; footprint Teensy_Footprint_Library:S8211-46R -> Package_DFN_QFN:DFN-8-1EP_3x3mm_P0.65mm_EP1.55x2.4mm; moved to F.Cu
- moved SDcard1 140.9 mm to (44.5, 33.5), turned to 180 degrees
- moved D1 120.3 mm to (229.9, 32.5), turned to 180 degrees
- moved MX1 99.2 mm to (235.2, 103.4), turned to 270 degrees
- moved C7 82.8 mm to (237.7, 70.1), turned to 90 degrees
- moved D6 78.6 mm to (99.1, 44.2), turned to 90 degrees
- moved R7 75.6 mm to (200.4, 117.9), turned to 270 degrees
- moved R2 71.6 mm to (140.2, 151.6), turned to 270 degrees
- moved R8 70.0 mm to (200.2, 91.9)
- moved D5 65.3 mm to (139.4, 144.0), turned to 180 degrees
- moved D4 63.4 mm to (127.0, 144.0), turned to 180 degrees
- moved R3 62.9 mm to (128.0, 151.6), turned to 270 degrees
- moved U1 61.7 mm to (192.3, 118.6)
- moved C3 61.2 mm to (127.0, 147.6), turned to 180 degrees
- moved C2 61.2 mm to (139.4, 147.6), turned to 180 degrees
- moved C4 52.8 mm to (102.6, 44.2), turned to 90 degrees
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Connections:
- C1 pad 1: IN1+ -> SusDipsFiltered-FR
- C1 pad 2: Net-(C1-Pad2) -> GND
- C10 pad 1: IN8+ -> GND
- C10 pad 2: Net-(C10-Pad2) -> +3V3
- C11 pad 1: Vinn_5V -> +5V
- C11 pad 2: Ground -> GND
- C2 pad 1: IN2+ -> SusDipsFiltered-FL
- C2 pad 2: Net-(C2-Pad2) -> GND
- C3 pad 1: Ground -> SusDipsFiltered-RR
- C3 pad 2: Vinn_5V -> GND
- C4 pad 1: IN3+ -> SusDipsFiltered-RL
- C4 pad 2: Net-(C4-Pad2) -> GND
- C5 pad 1: IN4+ -> ClutchPSFiltered
- C5 pad 2: Net-(C5-Pad2) -> GND
- C6 pad 1: IN5+ -> 12V_Ground
- C7 pad 1: IN6+ -> GND
- C7 pad 2: Net-(C7-Pad2) -> 12V_IN
- C8 pad 1: Ground -> GND
- C8 pad 2: Vinn_5V -> +3V3
- C9 pad 1: IN7+ -> +5V
- C9 pad 2: Net-(C9-Pad2) -> GND
- D1 pad 1: Out1 -> 12V_safe
- D1 pad 2: Ground -> Net-(D1-Pad2)
- D2 pad 1: Out2 -> ClutchPSFiltered
- D2 pad 2: Ground -> GND
- D3 pad 1: Out3 -> SusDipsFiltered-FR
- D3 pad 2: Ground -> GND
- D4 pad 1: Out4 -> SusDipsFiltered-RR
- D4 pad 2: Ground -> GND
- D5 pad 1: Out5 -> SusDipsFiltered-FL
- D5 pad 2: Ground -> GND
- D6 pad 1: Out6 -> SusDipsFiltered-RL
- D6 pad 2: Ground -> GND
- MX1 pad 10: 25_RX6_A11 -> VN-RX
- MX1 pad 11: 2_OUT2 -> 4G-RX
- MX1 pad 12: 3_LRCLK2 -> Net-(MX1-Pad12)
- MX1 pad 13: Ground -> Net-(MX1-Pad13)
- MX1 pad 14: 4_BCLK2 -> Servo-RX
- MX1 pad 15: 29_TX7 -> Servo-TX
- MX1 pad 16: 5_IN2 -> WSHE-RL
- MX1 pad 17: 28_RX7 -> Servo-IO
- MX1 pad 18: 6_OUT1D -> Net-(MX1-Pad18)
- MX1 pad 19: 33_MCLK2 -> CANFD-CANH
- MX1 pad 2: Vinn_5V -> GND
- MX1 pad 20: 7_RX2_OUT1A -> CANFD-CANL
- MX1 pad 21: 8_TX2_IN1 -> GearPS-MOSI
- MX1 pad 22: 32_OUT1B -> GearPS-MISO
- MX1 pad 23: 9_OUT1C -> Net-(MX1-Pad23)
- MX1 pad 24: 3V3 -> GearPS-CS
- MX1 pad 25: 26_A12 -> CAN2.0-CANH
- MX1 pad 26: Ground -> CAN2.0-CANL
- MX1 pad 27: Ground -> GearPS-SCK
- MX1 pad 28: Ground -> Net-(MX1-Pad28)
- MX1 pad 29: 21_RX3 -> Net-(MX1-Pad29)
- MX1 pad 3: Sensor_Input_1 -> Net-(MX1-Pad3)
- MX1 pad 30: 20_TX3 -> SusDips-FL
- MX1 pad 31: Sensor_Input_7 -> SusDips-RR
- MX1 pad 32: Sensor_Input_8 -> WSHE-FL
- MX1 pad 33: Sensor_Input_5 -> WSHE-FR
- MX1 pad 34: Sensor_Input_6 -> StearingAS
- MX1 pad 35: CANL -> WSHE-RR
- MX1 pad 36: CANH -> Net-(MX1-Pad36)
- MX1 pad 4: Sensor_Input_2 -> Net-(MX1-Pad4)
- MX1 pad 5: Sensor_Input_3 -> SusDips-RL
- MX1 pad 6: Sensor_Input_4 -> ClutchPS
- MX1 pad 7: 0_RX1 -> SusDips-FR
- MX1 pad 8: 24_TX6_A10 -> 4G-TX
- MX1 pad 9: 1_TX1 -> VN-TX
- PS1 pad 11: (no net) -> Net-(PS1-Pad11)
- PS1 pad 14: Vinn_5V -> +5V
- PS1 pad 16: Ground -> GND
- PS1 pad 2: Net-(PS1-Pad2) -> Net-(C6-Pad2)
- PS1 pad 22: Net-(D9-Pad1) -> 12V_safe
- PS1 pad 23: Net-(D9-Pad1) -> 12V_safe
- PS1 pad 3: Net-(PS1-Pad2) -> Net-(C6-Pad2)
- R1 pad 1: Sensor_Input_1 -> SusDipsFiltered-FR
- R1 pad 2: IN1+ -> SusDips-FR
- R2 pad 1: IN1+ -> SusDipsFiltered-FL
- R2 pad 2: Ground -> SusDips-FL
- R3 pad 1: Sensor_Input_2 -> SusDipsFiltered-RR
- R3 pad 2: IN2+ -> SusDips-RR
- R4 pad 1: IN2+ -> SusDipsFiltered-RL
- R4 pad 2: Ground -> SusDips-RL
- R5 pad 1: Sensor_Input_3 -> ClutchPS
- R5 pad 2: IN3+ -> ClutchPSFiltered
- R6 pad 1: IN3+ -> ClutchPSFiltered
- R6 pad 2: Ground -> GND
- R7 pad 1: Sensor_Input_4 -> CAN2.0-CANH
- R7 pad 2: IN4+ -> CAN2.0-CANL
- R8 pad 1: IN4+ -> CANFD-CANH
- R8 pad 2: Ground -> CANFD-CANL
- SDcard1 pad 1: (no net) -> Net-(SDcard1-Pad1)
- SDcard1 pad 2: 10_CS -> SD-CS
- SDcard1 pad 3: 11_MOSI -> SD-MOSI
- SDcard1 pad 4: 3.3V -> +3V3
- SDcard1 pad 5: 27_A13 -> SD-SCK
- SDcard1 pad 6: Ground -> GND
- SDcard1 pad 7: 12_MISO -> SD-MISO
- SDcard1 pad 8: (no net) -> Net-(SDcard1-Pad8)
- SDcard1 pad 9: Ground -> GND
- U1 pad 1: VBAT -> CAN2.0-TX
- U1 pad 2: VBAT -> GND
- U1 pad 3: Ground -> +5V
Routing:
- net GearPS-MOSI: track 0.00 -> 218.3 mm
- net WSHE-RR: track 0.00 -> 213.8 mm
- net +3V3: track 0.00 -> 207.0 mm
- net GearPS-MISO: track 0.00 -> 203.0 mm
- net StearingAS: track 0.00 -> 199.2 mm
- net WSHE-FL: track 0.00 -> 194.6 mm
- net WSHE-FR: track 0.00 -> 192.8 mm
- net Servo-IO: track 0.00 -> 184.0 mm
- net SusDips-RL: track 0.00 -> 170.8 mm
- net GearPS-CS: track 0.00 -> 163.3 mm
- net ClutchPS: track 0.00 -> 152.8 mm
- net WSHE-RL: track 0.00 -> 149.5 mm
- net SD-CS: track 0.00 -> 146.8 mm
- net SusDips-RR: track 0.00 -> 145.1 mm
- net CANFD-RX: track 0.00 -> 140.8 mm
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- removed copper zone on F.Cu, net Ground
- removed copper zone on B.Cu, net Vinn_5V
Other:
- board size 65 x 80 mm -> 255 x 155.7 mm
- board text removed: "1"
- board text removed: "2"
- board text removed: "T4AR20V2.0"

Commit message: Schematic DONE, started tracing
Parts:
- added H1: MountingHole, MountingHole:MountingHole_3.2mm_M3_ISO14580_Pad_TopBottom, F.Cu at (216.9, 111.3)
- added H2: MountingHole, MountingHole:MountingHole_3.2mm_M3_ISO14580_Pad_TopBottom, F.Cu at (57.9, 111.3)
- added H3: MountingHole, MountingHole:MountingHole_3.2mm_M3_ISO14580_Pad_TopBottom, F.Cu at (216.9, 33.3)
- added H4: MountingHole, MountingHole:MountingHole_3.2mm_M3_ISO14580_Pad_TopBottom, F.Cu at (57.9, 33.3)
- added U4: S8211-46R, Teensy_Footprint_Library:S8211-46R, B.Cu at (95.6, 72.5)
- D2, D3, D4, D5, D6: footprint Teensy_Footprint_Library:D_0603_MM3Z3V6T1G -> Teensy_Footprint_Library:D_SOD-323-MM3Z3V6T1G
- SDcard1: moved to B.Cu
- moved R8 276.7 mm to (-76.3, 79.4), turned to 0 degrees
- moved C2 201.1 mm to (-54.1, 92.8), turned to 0 degrees
- moved D3 198.5 mm to (-53.7, 108.9), turned to 0 degrees
- moved R1 195.4 mm to (-46.0, 97.8)
- moved D5 192.1 mm to (-49.4, 108.9), turned to 0 degrees
- moved R2 191.5 mm to (-42.0, 92.8), turned to 0 degrees
- moved C3 188.5 mm to (-54.1, 95.3), turned to 0 degrees
- moved C1 186.6 mm to (-42.0, 95.3), turned to 0 degrees
- moved R3 183.0 mm to (-46.0, 95.3), turned to 0 degrees
- moved D4 180.5 mm to (-49.4, 106.0), turned to 0 degrees
- moved C5 178.8 mm to (-54.1, 97.8), turned to 0 degrees
- moved D2 177.7 mm to (-53.7, 106.0), turned to 0 degrees
- moved R6 177.6 mm to (-50.1, 95.3), turned to 0 degrees
- moved R5 176.7 mm to (-46.0, 92.8), turned to 0 degrees
- moved R4 165.3 mm to (-50.1, 97.8)
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Connections:
- C6 pad 1: 12V_Ground -> GND
- C6 pad 2: Net-(C6-Pad2) -> +3V3
- C7 pad 1: GND -> (no net)
- C7 pad 2: 12V_IN -> 12V_safe
- MX1 pad 12: Net-(MX1-Pad12) -> (no net)
- MX1 pad 13: Net-(MX1-Pad13) -> (no net)
- MX1 pad 18: Net-(MX1-Pad18) -> (no net)
- MX1 pad 2: GND -> 12V_GND
- MX1 pad 23: Net-(MX1-Pad23) -> (no net)
- MX1 pad 28: Net-(MX1-Pad28) -> (no net)
- MX1 pad 29: Net-(MX1-Pad29) -> (no net)
- MX1 pad 3: Net-(MX1-Pad3) -> GND
- MX1 pad 36: Net-(MX1-Pad36) -> (no net)
- MX1 pad 4: Net-(MX1-Pad4) -> (no net)
- PS1 pad 11: Net-(PS1-Pad11) -> (no net)
- PS1 pad 2: Net-(C6-Pad2) -> 12V_GND
- PS1 pad 3: Net-(C6-Pad2) -> 12V_GND
- SDcard1 pad 1: Net-(SDcard1-Pad1) -> (no net)
- SDcard1 pad 8: Net-(SDcard1-Pad8) -> (no net)
- U2 pad CN11_16: (no net) -> +3V3
- U2 pad CN11_33: (no net) -> Net-(U2-PadCN11_33)
- U2 pad CN12_49: +3V3 -> (no net)
Routing:
- net GearPS-MOSI: track 218.3 -> 0.00 mm
- net GearPS-MISO: track 203.0 -> 0.00 mm
- net +3V3: track 207.0 -> 4.59 mm, vias 0 -> 1
- net StearingAS: track 199.2 -> 0.00 mm
- net WSHE-FL: track 194.6 -> 0.00 mm
- net WSHE-FR: track 192.8 -> 0.00 mm
- net Servo-IO: track 184.0 -> 0.00 mm
- net SusDips-RL: track 170.8 -> 0.00 mm
- net ClutchPS: track 152.8 -> 0.00 mm
- net WSHE-RL: track 149.5 -> 0.00 mm
- net SD-CS: track 146.8 -> 0.00 mm
- net SusDips-RR: track 145.1 -> 0.00 mm
- net CANFD-RX: track 140.8 -> 0.00 mm
- net WSHE-RR: track 213.8 -> 73.3 mm
- net CANFD-TX: track 139.3 -> 0.00 mm
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Other:
- board size 255 x 155.7 mm -> 167 x 86 mm
- net class Default: trace_width 0.25 -> 0.2; via_dia 0.8 -> 0.6; via_drill 0.4 -> 0.3
- rule trace_min: 0.25 -> 0.2
- rule via_min_size: 0.4 -> 0.6

Commit message: Trace V1.0 take 1
Parts:
- C1, C10, C11, C2, C3, C4, C5, C6, C8, C9, D2, D3, D4, D5, D6, R1, R2, R3, R4, R5, R6, R8, U3: moved to B.Cu
- moved R8 242.3 mm to (163.8, 111.8), turned to 90 degrees
- moved R4 192.1 mm to (141.8, 88.5)
- moved C4 188.1 mm to (138.0, 87.7), turned to 90 degrees
- moved D6 180.7 mm to (134.6, 87.5), turned to 90 degrees
- moved C3 179.4 mm to (121.7, 59.3), turned to 90 degrees
- moved C5 179.0 mm to (124.5, 84.9), turned to 90 degrees
- moved R6 178.0 mm to (127.6, 84.9), turned to 90 degrees
- moved C2 177.7 mm to (121.7, 66.2), turned to 90 degrees
- moved D2 176.1 mm to (121.1, 84.7), turned to 90 degrees
- moved R3 174.7 mm to (125.1, 60.1)
- moved D4 174.3 mm to (118.5, 59.3), turned to 90 degrees
- moved R5 173.7 mm to (127.6, 88.7), turned to 90 degrees
- moved D5 173.3 mm to (118.5, 66.1), turned to 90 degrees
- moved R2 169.3 mm to (125.3, 67.0)
- moved D3 164.7 mm to (109.5, 86.6), turned to 90 degrees
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Connections:
- C7 pad 1: (no net) -> 12V_GND
- MX1 pad 1: 12V_IN -> 4G-RX
- MX1 pad 10: VN-RX -> Servo-IO
- MX1 pad 11: 4G-RX -> GearPS-MISO
- MX1 pad 12: (no net) -> WSHE-RL
- MX1 pad 13: (no net) -> CANFD-CANH
- MX1 pad 14: Servo-RX -> CANFD-CANL
- MX1 pad 15: Servo-TX -> (no net)
- MX1 pad 16: WSHE-RL -> (no net)
- MX1 pad 17: Servo-IO -> (no net)
- MX1 pad 19: CANFD-CANH -> (no net)
- MX1 pad 2: 12V_GND -> VN-RX
- MX1 pad 20: CANFD-CANL -> (no net)
- MX1 pad 21: GearPS-MOSI -> ClutchPS
- MX1 pad 22: GearPS-MISO -> SusDips-RL
- MX1 pad 23: (no net) -> SusDips-FR
- MX1 pad 24: GearPS-CS -> GearPS-SCK
- MX1 pad 25: CAN2.0-CANH -> SusDips-FL
- MX1 pad 26: CAN2.0-CANL -> SusDips-RR
- MX1 pad 27: GearPS-SCK -> +5V
- MX1 pad 28: (no net) -> WSHE-FL
- MX1 pad 29: (no net) -> WSHE-FR
- MX1 pad 3: GND -> VN-TX
- MX1 pad 30: SusDips-FL -> StearingAS
- MX1 pad 31: SusDips-RR -> GearPS-CS
- MX1 pad 32: WSHE-FL -> WSHE-RR
- MX1 pad 33: WSHE-FR -> CAN2.0-CANL
- MX1 pad 34: StearingAS -> CAN2.0-CANH
- MX1 pad 35: WSHE-RR -> 12V_GND
- MX1 pad 36: (no net) -> 12V_IN
- MX1 pad 4: (no net) -> 4G-TX
- MX1 pad 5: SusDips-RL -> GND
- MX1 pad 6: ClutchPS -> Servo-RX
- MX1 pad 7: SusDips-FR -> Servo-TX
- MX1 pad 8: 4G-TX -> +3V3
- MX1 pad 9: VN-TX -> GearPS-MOSI
- U2 pad CN11_72: (no net) -> GND
- Z1 pad 2: GND -> 12V_GND
Routing:
- net GND: track 0.00 -> 780.8 mm, vias 0 -> 4
- net +5V: track 0.00 -> 366.1 mm, vias 0 -> 5
- net +3V3: track 4.59 -> 368.2 mm, vias 1 -> 5
- net 4G-RX: track 0.00 -> 144.8 mm
- net VN-RX: track 0.00 -> 139.2 mm
- net SD-MOSI: track 0.00 -> 138.9 mm
- net VN-TX: track 0.00 -> 134.9 mm
- net 4G-TX: track 0.00 -> 132.5 mm
- net Servo-RX: track 0.00 -> 125.4 mm
- net GearPS-SCK: track 0.00 -> 125.3 mm, vias 0 -> 1
- net Servo-TX: track 0.00 -> 123.0 mm
- net CAN2.0-CANH: track 0.00 -> 121.8 mm
- net CAN2.0-CANL: track 0.00 -> 120.5 mm
- net WSHE-FL: track 0.00 -> 110.7 mm
- net SD-MISO: track 0.00 -> 110.3 mm
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Other:
- board text added: "AR21"
- board text added: "Battery"
- board text added: "CAN2.0"
- board text added: "CANFD"

Commit message: Small fixes. Not done yet
Parts:
- moved C2 29.7 mm to (151.3, 67.1)
- moved D5 29.7 mm to (148.2, 67.0)
- moved R2 29.7 mm to (155.0, 67.9)
- moved C3 29.7 mm to (151.3, 60.4)
- moved D4 29.7 mm to (148.2, 60.3)
- moved R3 29.7 mm to (154.7, 61.2)
- moved SDcard1 19.0 mm to (71.6, 80.3), turned to 270 degrees
- moved C6 12.4 mm to (75.7, 73.8), turned to 90 degrees
- moved U4 6.18 mm to (90.0, 71.8)
Routing:
- net GND: track 780.8 -> 632.5 mm
- net SusDips-RR: track 83.9 -> 53.8 mm
- net SusDips-FL: track 81.3 -> 51.2 mm
- net SusDipsFiltered-RR: track 29.0 -> 58.4 mm
- net SusDipsFiltered-FL: track 38.8 -> 68.3 mm
- net SD-MOSI: track 138.9 -> 123.7 mm
- net Net-(U2-PadCN11_33): track 41.4 -> 47.4 mm
- net SD-MISO: track 110.3 -> 115.4 mm
- net SD-SCK: track 109.2 -> 106.1 mm
- net +3V3: track 368.2 -> 365.4 mm
- net 12V_GND: track 93.8 -> 95.4 mm
- net SD-CS: track 98.6 -> 100.0 mm, vias 0 -> 2
- net +5V: track 366.1 -> 365.7 mm, vias 5 -> 6

Commit message: Finished PCB V1.0? Added 6 more pins
Parts:
- moved R7 1.26 mm to (116.9, 33.4)
Connections:
- MX1 pad 15: (no net) -> I2C1-SDA
- MX1 pad 16: (no net) -> ClutchPS
- MX1 pad 17: (no net) -> SusDips-RL
- MX1 pad 18: (no net) -> SusDips-FR
- MX1 pad 19: (no net) -> GearPS-SCK
- MX1 pad 20: (no net) -> SusDips-FL
- MX1 pad 21: ClutchPS -> SusDips-RR
- MX1 pad 22: SusDips-RL -> +5V
- MX1 pad 23: SusDips-FR -> WSHE-FL
- MX1 pad 24: GearPS-SCK -> WSHE-FR
- MX1 pad 25: SusDips-FL -> StearingAS
- MX1 pad 26: SusDips-RR -> GearPS-CS
- MX1 pad 27: +5V -> WSHE-RR
- MX1 pad 28: WSHE-FL -> GPIO-digital2
- MX1 pad 29: WSHE-FR -> GPIO-analog-ut2
- MX1 pad 30: StearingAS -> GPIO-analog-ut1
- MX1 pad 31: GearPS-CS -> GPIO-digital1
- MX1 pad 32: WSHE-RR -> CAN2.0-CANL
- MX1 pad 33: CAN2.0-CANL -> CAN2.0-CANH
- MX1 pad 34: CAN2.0-CANH -> I2C1-SCL
- U2 pad CN11_21: (no net) -> I2C1-SDA
- U2 pad CN12_22: (no net) -> GPIO-digital1
- U2 pad CN12_3: (no net) -> I2C1-SCL
- U2 pad CN12_50: (no net) -> GPIO-analog-ut1
- U2 pad CN12_60: (no net) -> GPIO-analog-ut2
- U2 pad CN12_62: (no net) -> GPIO-digital2
- U2 pad CN12_72: (no net) -> GND
Routing:
- net I2C1-SCL: track 0.00 -> 144.6 mm
- net GPIO-digital1: track 0.00 -> 114.0 mm
- net I2C1-SDA: track 0.00 -> 107.8 mm, vias 0 -> 1
- net GPIO-analog-ut1: track 0.00 -> 77.8 mm
- net GPIO-analog-ut2: track 0.00 -> 64.5 mm
- net GPIO-digital2: track 0.00 -> 62.0 mm
- net +5V: track 365.7 -> 378.4 mm
- net 12V_IN: track 31.3 -> 36.4 mm
- net StearingAS: track 93.7 -> 98.1 mm
- net WSHE-FL: track 110.7 -> 115.0 mm
- net WSHE-FR: track 102.3 -> 106.6 mm
- net GearPS-CS: track 85.9 -> 90.0 mm
- net WSHE-RR: track 80.6 -> 84.4 mm
- net SusDips-RR: track 53.8 -> 56.1 mm
- net SusDips-FR: track 90.3 -> 88.1 mm
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- added copper zone on B.Cu, net GND

Commit message: A slight Adjustment
Routing:
- net GND: track 630.6 -> 602.8 mm, vias 4 -> 7
- net +5V: track 378.4 -> 376.5 mm, vias 6 -> 5
