File: AR20_Pedalbox/Pedal_pcb/Pedalbox Extenion Board/Pedalbox Extenion Board.kicad_pcb (KiCad board)
At the start: 2 copper layers, 41 x 37.2 mm, 24 parts, among them P1 MX23A18NF1, U1 ACM_2020, U2 L78L05_SO8, U3 L78L05_SO8

Commit message: Updated iBOM
Parts:
- C5, C6, C8, C9: value C_Small -> 0,1uF
- R2, R5: value R_Small -> 7,5K
- R4: value R_Small -> 15K
- renumbered R1 to 15K1
