File: AR20_Pedalbox/Pedal_pcb/Pedalbox Extenion Board/Pedalbox Extenion Board.sch (KiCad schematic (older format))
At the start: 4 parts, among them P1 MX23A12NF1, U1 ACM_2020, U2 L78L05_SO8, U3 L78L05_SO8

Commit message: Started on PCB layout and added 18pin connector
Parts:
- removed P1: MX23A12NF1, Pedalbox Extenion Board:JAE_MX23A12NF1, symbol Pedalbox~Extenion~Board:MX23A12NF1
- added C1, C3: 0.33uF, Capacitor_SMD:C_0603_1608Metric, symbol Device:C_Small
- added C2, C4: 0.1uF, Capacitor_SMD:C_0603_1608Metric, symbol Device:C_Small
- added P1: MX23A18NF1, MX23A18NF1:JAE_MX23A18NF1, symbol ACM_2020_Symbol:MX23A18NF1
Connections:
- net labels added: APPS1_GND, APPS1_Signal, APPS1_Supply, APPS2_GND, APPS2_Signal, APPS2_Supply, BPS1_Signal, BPS2_GND, BPS2_Signal, BPS2_Supply, CANH, CANL, Steering_Angle_Sensor_GND, Steering_Angle_Sensor_Signal, Steering_Angle_Sensor_Supply
- wire segments 4 -> 36
Other:
- note added: "Redundant 2x 100mA LDO for APPS sensors"
- note removed: "Redundant LDO for APPS sensors"
- moved on the sheet: U1, U2, U3

Commit message: Pedalbox PCB Ready - Just need some more silkscreen... ;)
Parts:
- added C5, C6, C7, C8, C9: C_Small, Capacitor_SMD:C_0603_1608Metric_Pad1.05x0.95mm_HandSolder, symbol Device:C_Small
- added H1: MountingHole, MountingHole:MountingHole_2.2mm_M2, symbol Mechanical:MountingHole
- added R1, R2, R3, R4, R5: R_Small, Resistor_SMD:R_0603_1608Metric_Pad1.05x0.95mm_HandSolder, symbol Device:R_Small
- added R10, R6, R7, R8, R9: 4K7, Resistor_SMD:R_0603_1608Metric_Pad1.05x0.95mm_HandSolder, symbol Device:R_Small
- C1, C2, C3, C4: footprint Capacitor_SMD:C_0603_1608Metric -> Capacitor_SMD:C_0603_1608Metric_Pad1.05x0.95mm_HandSolder
Connections:
- net BPS2_GND is gone; now on net Steering_Angle_Sensor_Signal: P1.9
- net BPS2_Supply is gone; now on net BPS1_Signal: P1.8
- net +12V: now also P1.6; no longer P1.1
- net +5V: now also P1.13, P1.14; no longer P1.12, P1.5
- net APPS1_Signal: now also P1.2, R1.2; no longer P1.18, U1.3 (15/A1-PC1)
- net APPS1_Supply: now also P1.1; no longer P1.16
- net APPS2_Signal: now also P1.3, R4.2; no longer P1.15, U1.2 (16/A2-PC2)
- net APPS2_Supply: now also P1.10; no longer P1.13
- net BPS1_Signal: now also R2.2; no longer P1.11
- net BPS2_Signal: now also P1.7, R5.2; no longer P1.10
- net CANH: now also P1.4; no longer P1.3
- net CANL: now also P1.5; no longer P1.4
- net GND: now also P1.11, P1.12, P1.15, P1.16, P1.18, C5.2, C6.2, C7.2, C8.2, C9.2, R10.2, R6.2, R7.2, R8.2, R9.2; no longer P1.14, P1.2, P1.6
- net Steering_Angle_Sensor_Signal: now also R3.2; no longer P1.7, U1.1 (14/A0-PC0)
- net BPS1_Signal_Filtered: now reaches U1.4 (17/A3-PC3)
- net BPS1_Signal_Filtered: now also C6.1, R2.1, R6.1
- net BPS2_Signal_Filtered: now reaches U1.6 (18/A4-PC4)
- net BPS2_Signal_Filtered: now also C9.1, R10.1, R5.1
- new net APPS1_Signal_Filtered: C5.1, R1.1, R7.1, U1.1 (14/A0-PC0)
- new net APPS2_Signal_Filtered: C8.1, R4.1, R9.1, U1.3 (15/A1-PC1)
- new net Steering_Angle_Sensor_Signal_Filtered: C7.1, R3.1, R8.1, U1.2 (16/A2-PC2)
Other:
- note added: "Cutoff [Hz]:\nTime Constant:\n"
- note added: "Low pass filter for APPS1"
- note added: "Low pass filter for APPS2"
- note added: "Low pass filter for BPS1"
- note added: "Low pass filter for BPS2"
- note added: "Low pass filter for SAS"
- note added: "Mechanical Mouting"
- moved on the sheet: C1, C2, C3, C4, P1, U1, U2, U3

Commit message: Fixed traces, changed ACM footprint and generated gerber
Parts:
- U1: footprint Pedalbox Extenion Board:ACM_2020_Footprint -> Pedalbox Extenion Board:ACM_2020_Footprint_wo_silk
Changed lines of the file:
@@
 F 0 "U1" H 9250 8765 50  0000 C CNN
 F 1 "ACM_2020" H 9250 8674 50  0000 C CNN
-F 2 "Pedalbox Extenion Board:ACM_2020_Footprint" H 9225 6200 50  0001 C CNN
+F 2 "Pedalbox Extenion Board:ACM_2020_Footprint_wo_silk" H 9225 6200 50  0001 C CNN
 F 3 "" H 9225 6200 50  0001 C CNN
 	1    9225 6200

Commit message: Set filtering values
Parts:
- 15K: renamed from R1; symbol Device:R_Small -> Pedalbox-Extenion-Board-rescue:R_Small-Device
- C1, C2, C3, C4, C7: symbol Device:C_Small -> Pedalbox-Extenion-Board-rescue:C_Small-Device
- C5, C6, C8, C9: value C_Small -> 0,1uF; symbol Device:C_Small -> Pedalbox-Extenion-Board-rescue:C_Small-Device
- H1: symbol Mechanical:MountingHole -> Pedalbox-Extenion-Board-rescue:MountingHole-Mechanical
- R10, R3, R6, R7, R8, R9: symbol Device:R_Small -> Pedalbox-Extenion-Board-rescue:R_Small-Device
- R2, R5: value R_Small -> 7,5K; symbol Device:R_Small -> Pedalbox-Extenion-Board-rescue:R_Small-Device
- R4: value R_Small -> 15K; symbol Device:R_Small -> Pedalbox-Extenion-Board-rescue:R_Small-Device
- U2, U3: symbol Regulator_Linear:L78L05_SO8 -> Pedalbox-Extenion-Board-rescue:L78L05_SO8-Regulator_Linear
Changed lines of the file:
@@
 EESchema Schematic File Version 4
-LIBS:Pedalbox Extenion Board-cache
-EELAYER 29 0
+EELAYER 30 0
 EELAYER END
 $Descr A4 11693 8268
@@
 $EndComp
 $Comp
-L power:GND #PWR0101
+L Pedalbox-Extenion-Board-rescue:GND-power #PWR0101
 U 1 1 5E288B46
 P 10025 3900
@@
 $EndComp
 $Comp
-L power:GND #PWR0102
+L Pedalbox-Extenion-Board-rescue:GND-power #PWR0102
 U 1 1 5E289D7E
 P 10025 4200
@@
 $EndComp
 $Comp
-L power:GND #PWR0103
+L Pedalbox-Extenion-Board-rescue:GND-power #PWR0103
 U 1 1 5E28A22E
 P 10025 4350
@@
 $EndComp
 $Comp
-L power:GND #PWR0104
+L Pedalbox-Extenion-Board-rescue:GND-power #PWR0104
 U 1 1 5E28A518
 P 10025 4650
@@
 $EndComp
 $Comp
-L power:+12V #PWR0105
+L Pedalbox-Extenion-Board-rescue:+12V-power #PWR0105
 U 1 1 5E28AA01
 P 10325 5950
@@
 	10325 6000 10325 5950
 $Comp
-L power:GND #PWR0106
+L Pedalbox-Extenion-Board-rescue:GND-power #PWR0106
 U 1 1 5E28BEB2
 P 8475 5100
@@
 $EndComp
 $Comp
-L power:+5V #PWR0107
+L Pedalbox-Extenion-Board-rescue:+5V-power #PWR0107
 U 1 1 5E28C9C6
 P 10450 5075
@@
 What need to be implemented:\n- Redundant APPS out with redundant LDO\n- Pull down resistors for sensor inputs\n-
 $Comp
-L Regulator_Linear:L78L05_SO8 U2
+L Pedalbox-Extenion-Board-rescue:L78L05_SO8-Regulator_Linear U2
 U 1 1 5E28F187
 P 1750 1775
@@
 $EndComp
 $Comp
-L Regulator_Linear:L78L05_SO8 U3
+L Pedalbox-Extenion-Board-rescue:L78L05_SO8-Regulator_Linear U3
 U 1 1 5E290B0E
 P 3700 1775
@@
 $EndComp
 $Comp
-L Device:C_Small C3
+L Pedalbox-Extenion-Board-rescue:C_Small-Device C3
 U 1 1 5E29DD14
 P 3300 2000
@@
 $EndComp
 $Comp
-L Device:C_Small C4
+L Pedalbox-Extenion-Board-rescue:C_Small-Device C4
 U 1 1 5E2A8BE8
 P 4075 2000
@@
 $EndComp
 $Comp
-L Device:C_Small C1
+L Pedalbox-Extenion-Board-rescue:C_Small-Device C1
 U 1 1 5E2B118B
 P 1325 2025
@@
 $EndComp
 $Comp
-L Device:C_Small C2
+L Pedalbox-Extenion-Board-rescue:C_Small-Device C2
 U 1 1 5E2B1B66
 P 2100 2075
@@
 $EndComp
 $Comp
-L power:GND #PWR0108
+L Pedalbox-Extenion-Board-rescue:GND-power #PWR0108
 U 1 1 5E2B26A0
 P 3700 2075
@@
 $EndComp
 $Comp
-L power:GND #PWR0109
+L Pedalbox-Extenion-Board-rescue:GND-power #PWR0109
 U 1 1 5E2B36B2
 P 1750 2075
@@
 $EndComp
 $Comp
-L power:GND #PWR0110
+L Pedalbox-Extenion-Board-rescue:GND-power #PWR0110
 U 1 1 5E2B3EFC
 P 2100 2175
@@
 $EndComp
 $Comp
-L power:GND #PWR0111
+L Pedalbox-Extenion-Board-rescue:GND-power #PWR0111
 U 1 1 5E2B436A
 P 1325 2125
@@
 $EndComp
 $Comp
-L power:GND #PWR0112
+L Pedalbox-Extenion-Board-rescue:GND-power #PWR0112
 U 1 1 5E2B4912
 P 3300 2100
@@
 $EndComp
 $Comp
-L power:GND #PWR0113
+L Pedalbox-Extenion-Board-rescue:GND-power #PWR0113
 U 1 1 5E2B4D8C
 P 4075 2100
@@
 $EndComp
 $Comp
-L power:+12V #PWR0114
+L Pedalbox-Extenion-Board-rescue:+12V-power #PWR0114
 U 1 1 5E2B8DAF
 P 2825 3575
@@
 CANL
 $Comp
-L power:+12V #PWR0116
+L Pedalbox-Extenion-Board-rescue:+12V-power #PWR0116
 U 1 1 5E2BCE59
 P 1325 1675
@@
 $EndComp
 $Comp
-L power:+12V #PWR0117
+L Pedalbox-Extenion-Board-rescue:+12V-power #PWR0117
 U 1 1 5E2BD83E
 P 3300 1600
@@
 CANL
 $Comp
-L power:+5V #PWR0118
+L Pedalbox-Extenion-Board-rescue:+5V-power #PWR0118
 U 1 1 5E2CD018
 P 10450 5675
@@
 	10450 5700 10450 5675
 $Comp
-L power:+5V #PWR0119
+L Pedalbox-Extenion-Board-rescue:+5V-power #PWR0119
 U 1 1 5E2CD86D
 P 10450 5375
@@
 BPS2_Signal
 $Comp
-L power:+5V #PWR0120
+L Pedalbox-Extenion-Board-rescue:+5V-power #PWR0120
 U 1 1 5E2D4FDA
 P 4625 3450
@@
 	4625 3475 3975 3475
 $Comp
-L power:GND #PWR0123
+L Pedalbox-Extenion-Board-rescue:GND-power #PWR0123
 U 1 1 5E2DE5D8
 P 4100 3925
@@
 APPS1_Signal
 $Comp
-L Device:R_Small R1
+L Pedalbox-Extenion-Board-rescue:R_Small-Device 15K
 U 1 1 5E33B337
 P 1650 4700
-F 0 "R1" V 1454 4700 50  0000 C CNN
+F 0 "15K" V 1454 4700 50  0000 C CNN
 F 1 "R_Small" V 1545 4700 50  0000 C CNN
 F 2 "Resistor_SMD:R_0603_1608Metric_Pad1.05x0.95mm_HandSolder" H 1650 4700 50  0001 C CNN
@@
 $EndComp
 $Comp
-L Device:C_Small C5
+L Pedalbox-Extenion-Board-rescue:C_Small-Device C5
 U 1 1 5E33C741
 P 1900 5000
 F 0 "C5" H 1675 5025 50  0000 L CNN
-F 1 "C_Small" H 1475 4925 50  0000 L CNN
+F 1 "0,1uF" H 1475 4925 50  0000 L CNN
 F 2 "Capacitor_SMD:C_0603_1608Metric_Pad1.05x0.95mm_HandSolder" H 1900 5000 50  0001 C CNN
 F 3 "~" H 1900 5000 50  0001 C CNN
@@
 	1900 4700 1900 4900
 $Comp
-L power:GND #PWR0125
+L Pedalbox-Extenion-Board-rescue:GND-power #PWR0125
 U 1 1 5E33EE5F
 P 1900 5100
@@
 APPS2_Signal
 $Comp
-L Device:R_Small R4
+L Pedalbox-Extenion-Board-rescue:R_Small-Device R4
 U 1 1 5E347142
 P 4475 4700
 F 0 "R4" V 4279 4700 50  0000 C CNN
-F 1 "R_Small" V 4370 4700 50  0000 C CNN
+F 1 "15K" V 4370 4700 50  0000 C CNN
 F 2 "Resistor_SMD:R_0603_1608Metric_Pad1.05x0.95mm_HandSolder" H 4475 4700 50  0001 C CNN
 F 3 "~" H 4475 4700 50  0001 C CNN
@@
 $EndComp
 $Comp
-L Device:C_Small C8
+L Pedalbox-Extenion-Board-rescue:C_Small-Device C8
 U 1 1 5E347148
 P 4725 5000
 F 0 "C8" H 4375 5000 50  0000 L CNN
-F 1 "C_Small" H 4350 4925 50  0000 L CNN
+F 1 "0,1uF" H 4350 4925 50  0000 L CNN
 F 2 "Capacitor_SMD:C_0603_1608Metric_Pad1.05x0.95mm_HandSolder" H 4725 5000 50  0001 C CNN
 F 3 "~" H 4725 5000 50  0001 C CNN
@@
 	4725 4700 4725 4900
 $Comp
-L power:GND #PWR0126
+L Pedalbox-Extenion-Board-rescue:GND-power #PWR0126
 U 1 1 5E347151
 P 4725 5100
@@
 Low pass filter for BPS1
 $Comp
-L Device:R_Small R2
+L Pedalbox-Extenion-Board-rescue:R_Small-Device R2
 U 1 1 5E352686
 P 1675 5875
 F 0 "R2" V 1479 5875 50  0000 C CNN
-F 1 "R_Small" V 1570 5875 50  0000 C CNN
+F 1 "7,5K" V 1570 5875 50  0000 C CNN
 F 2 "Resistor_SMD:R_0603_1608Metric_Pad1.05x0.95mm_HandSolder" H 1675 5875 50  0001 C CNN
 F 3 "~" H 1675 5875 50  0001 C CNN
@@
 $EndComp
 $Comp
-L Device:C_Small C6
+L Pedalbox-Extenion-Board-rescue:C_Small-Device C6
 U 1 1 5E35268C
 P 1925 6175
 F 0 "C6" H 1675 6200 50  0000 L CNN
-F 1 "C_Small" H 1575 6125 50  0000 L CNN
+F 1 "0,1uF" H 1575 6125 50  0000 L CNN
 F 2 "Capacitor_SMD:C_0603_1608Metric_Pad1.05x0.95mm_HandSolder" H 1925 6175 50  0001 C CNN
 F 3 "~" H 1925 6175 50  0001 C CNN
@@
 	1925 5875 1925 6075
 $Comp
-L power:GND #PWR0127
+L Pedalbox-Extenion-Board-rescue:GND-power #PWR0127
 U 1 1 5E352695
 P 1925 6275
@@
 Low pass filter for BPS2
 $Comp
-L Device:R_Small R5
+L Pedalbox-Extenion-Board-rescue:R_Small-Device R5
 U 1 1 5E3526A4
 P 4500 5875
 F 0 "R5" V 4304 5875 50  0000 C CNN
-F 1 "R_Small" V 4395 5875 50  0000 C CNN
+F 1 "7,5K" V 4395 5875 50  0000 C CNN
 F 2 "Resistor_SMD:R_0603_1608Metric_Pad1.05x0.95mm_HandSolder" H 4500 5875 50  0001 C CNN
 F 3 "~" H 4500 5875 50  0001 C CNN
@@
 $EndComp
 $Comp
-L Device:C_Small C9
+L Pedalbox-Extenion-Board-rescue:C_Small-Device C9
 U 1 1 5E3526AA
 P 4750 6175
 F 0 "C9" H 4550 6200 50  0000 L CNN
-F 1 "C_Small" H 4425 6125 50  0000 L CNN
+F 1 "0,1uF" H 4425 6125 50  0000 L CNN
 F 2 "Capacitor_SMD:C_0603_1608Metric_Pad1.05x0.95mm_HandSolder" H 4750 6175 50  0001 C CNN
 F 3 "~" H 4750 6175 50  0001 C CNN
@@
 	4750 5875 4750 6075
 $Comp
-L power:GND #PWR0128
+L Pedalbox-Extenion-Board-rescue:GND-power #PWR0128
 U 1 1 5E3526B3
 P 4750 6275
@@
 Low pass filter for SAS
 $Comp
-L Device:R_Small R3
+L Pedalbox-Extenion-Board-rescue:R_Small-Device R3
 U 1 1 5E35DDAD
 P 2375 7025
@@
 $EndComp
 $Comp
-L Device:C_Small C7
+L Pedalbox-Extenion-Board-rescue:C_Small-Device C7
 U 1 1 5E35DDB3
 P 2625 7325
@@
 	2625 7025 2625 7225
 $Comp
-L power:GND #PWR0129
+L Pedalbox-Extenion-Board-rescue:GND-power #PWR0129
 U 1 1 5E35DDBC
 P 2625 7425
@@
 BPS1_Signal_Filtered
 $Comp
-L Device:R_Small R9
+L Pedalbox-Extenion-Board-rescue:R_Small-Device R9
 U 1 1 5E36DE4D
 P 4950 4875
@@
 $EndComp
 $Comp
-L power:GND #PWR04
+L Pedalbox-Extenion-Board-rescue:GND-power #PWR04
 U 1 1 5E36F8A4
 P 4950 4975
@@
 $EndComp
 $Comp
-L Device:R_Small R7
+L Pedalbox-Extenion-Board-rescue:R_Small-Device R7
 U 1 1 5E372C45
 P 2150 4850
@@
 $EndComp
 $Comp
-L power:GND #PWR02
+L Pedalbox-Extenion-Board-rescue:GND-power #PWR02
 U 1 1 5E372C4B
 P 2150 4950
@@
 $EndComp
 $Comp
-L Device:R_Small R6
+L Pedalbox-Extenion-Board-rescue:R_Small-Device R6
 U 1 1 5E374451
 P 2125 6025
@@
 $EndComp
 $Comp
-L power:GND #PWR01
+L Pedalbox-Extenion-Board-rescue:GND-power #PWR01
 U 1 1 5E374457
 P 2125 6125
@@
 $EndComp
 $Comp
-L Device:R_Small R10
+L Pedalbox-Extenion-Board-rescue:R_Small-Device R10
 U 1 1 5E376179
 P 4975 6025
@@
 $EndComp
 $Comp
-L power:GND #PWR05
+L Pedalbox-Extenion-Board-rescue:GND-power #PWR05
 U 1 1 5E37617F
 P 4975 6125
@@
 $EndComp
 $Comp
-L Device:R_Small R8
+L Pedalbox-Extenion-Board-rescue:R_Small-Device R8
 U 1 1 5E3783E9
 P 2875 7200
@@
 $EndComp
 $Comp
-L power:GND #PWR03
+L Pedalbox-Extenion-Board-rescue:GND-power #PWR03
 U 1 1 5E3783EF
 P 2875 7300
@@
 Connection ~ 3975 3875
 $Comp
-L power:GND #PWR0130
+L Pedalbox-Extenion-Board-rescue:GND-power #PWR0130
 U 1 1 5E43BCCD
 P 4225 3250
@@
 Connection ~ 3975 3475
 $Comp
-L Mechanical:MountingHole H1
+L Pedalbox-Extenion-Board-rescue:MountingHole-Mechanical H1
 U 1 1 5E460860
 P 5700 7075

Commit message: Updated iBOM
Parts:
- renumbered 15K to 15K1
Changed lines of the file:
@@
 APPS1_Signal
 $Comp
-L Pedalbox-Extenion-Board-rescue:R_Small-Device 15K
+L Pedalbox-Extenion-Board-rescue:R_Small-Device 15K1
 U 1 1 5E33B337
 P 1650 4700
-F 0 "15K" V 1454 4700 50  0000 C CNN
+F 0 "15K1" V 1454 4700 50  0000 C CNN
 F 1 "R_Small" V 1545 4700 50  0000 C CNN
 F 2 "Resistor_SMD:R_0603_1608Metric_Pad1.05x0.95mm_HandSolder" H 1650 4700 50  0001 C CNN
